File: MC8P_MIDI_CONTROLLER_KiCad/MC8P_MIDI_CONTROLLER/MC8P_MIDI_CONTROLLER.kicad_sch (KiCad schematic)
At the start: 34 parts, among them J1 MIDI OUT, J2 5V, SW1 ASSIGN, SW2 ENTER, SW3 PREV, SW4 NEXT, U1 Teensy4.0

Commit message: Black Pill Schematic & PCB
Parts:
- removed C12: 10uF_4x5.3_10V, Capacitor_THT:CP_Radial_D4.0mm_P1.50mm, symbol PCM_4ms_Capacitor:10uF_4x5.3_10V
- removed J2: 5V, Connector_BarrelJack:BarrelJack_GCT_DCJ200-10-A_Horizontal, symbol Connector:Barrel_Jack_MountingPin
- removed U1: Teensy4.0, teensy:Teensy40, symbol teensy:Teensy4.0
- added C12, C13, C14, C15: 100nF_0603_16V, Capacitor_SMD:C_1206_3216Metric, symbol PCM_4ms_Capacitor:100nF_0603_16V
- added C16: 10uF, Capacitor_SMD:C_1206_3216Metric_Pad1.33x1.80mm_HandSolder, symbol Device:C
- added D1: LED, LED_SMD:LED_1206_3216Metric_Pad1.42x1.75mm_HandSolder, symbol Device:LED
- added D2: BAT43, Diode_SMD:D_SOD-123, symbol PCM_Diode_Schottky_AKL:BAT43
- added F1: 1A_15V, Fuse:Fuse_1812_4532Metric, symbol PCM_4ms_Regulator:Polyfuse_3A_15V
- added J2: Jack-DC, Connector_BarrelJack:BarrelJack_GCT_DCJ200-10-A_Horizontal, symbol Connector:Jack-DC
- added R7, R8: 10k_0402, PCM_4ms_Resistor:R_0603, symbol PCM_4ms_Resistor:10k_0402
- added U1: ~, blackpill:Z_module_black_pill_STM32F411, symbol STM32F411CEU6_BlackPill:BlackPill_STM32F411CEU6
- added U3: CD74HC4067M, Package_SO:SOIC-24W_7.5x15.4mm_P1.27mm, symbol 74xx:CD74HC4067M
- added U4: W25Q64, Package_SO:SOIC-8_3.9x4.9mm_P1.27mm, symbol W25Q64_SPI_FLASH:W25Q64
- C1, C2, C3, C4, C5, C6, C7, C8: footprint Capacitor_THT:C_Axial_L3.8mm_D2.6mm_P7.50mm_Horizontal -> Capacitor_SMD:C_1206_3216Metric_Pad1.33x1.80mm_HandSolder
- C10, C9: footprint Capacitor_THT:C_Disc_D5.0mm_W2.5mm_P5.00mm -> Capacitor_SMD:C_1206_3216Metric_Pad1.33x1.80mm_HandSolder
- R1, R2, R3, R4: footprint PCM_4ms_Resistor:R_Axial_DIN0207_L6.3mm_D2.5mm_P7.62mm_Horizontal -> PCM_4ms_Resistor:R_0603
- R5, R6: footprint PCM_4ms_Resistor:R_Axial_DIN0207_L6.3mm_D2.5mm_P7.62mm_Horizontal -> PCM_4ms_Resistor:R_0603; Display 220R -> 33R
- renumbered SSD1 to SSD1306
Connections:
- net 3V3: now also R6.1, C12.2, C13.1, C14.2, D1.2 (A), U1.20 (3V3), U1.38 (3V3), U3.24 (VCC), U4.3 (WP), U4.7 (HOLD), U4.8 (VCC)
- net GND: now also C12.1, C13.2, C14.1, C15.1, C16.2, J2.2, R7.2, U1.19 (GND), U1.39 (GND), U3.12 (GND), U4.4 (GND)
- net SCL0: now also U1.14 (PB6/SCL1/TX1)
- net SDA0: now also U1.15 (PB7/SDA1/RX1)
- net TX0: now also U1.28 (PA2/ADC2/TX2)
- net Vcc: now also D2.1 (K), U1.18 (5V), U1.40 (5V); no longer R6.1
- net A0 renamed pot1
- net pot1: now also U3.9 (I0)
- net A1 renamed pot2
- net pot2: now also U3.8 (I1)
- net A2 renamed pot3
- net pot3: now also U3.7 (I2)
- net A3 renamed pot4
- net pot4: now also U3.6 (I3)
- net A6 renamed pot5
- net pot5: now also C5.1, U3.5 (I4); no longer C8.1
- net A7 renamed pot6
- net pot6: now also C6.1, U3.4 (I5); no longer C7.1
- net A8 renamed pot7
- net pot7: now also C7.1, U3.3 (I6); no longer C6.1
- net A9 renamed pot8
- net pot8: now also C8.1, U3.2 (I7); no longer C5.1
- net D5 renamed ASSIGN
- net ASSIGN: now also U1.1 (PB12/SCK3)
- net D6 renamed ENTER
- net ENTER: now also U1.2 (PB13/SCK4)
- net D7 renamed PREV
- net PREV: now also U1.3 (PB14/MISO2)
- net D8 renamed NEXT
- net NEXT: now also U1.4 (PB15/MOSI2)
- new net: R7.1, U3.15 (~{E})
- new net: C15.2, C16.1, D2.2 (A), F1.2
- new net: D1.1 (K), R8.2
- new net: F1.1, J2.1
- new net CLK: U1.31 (PA5/ADC5/SCK1), U4.6 (CLK)
- new net CS: R8.1, U1.30 (PA4/ADC4), U4.1 (CS)
- new net MISO: U1.32 (PA6/ADC6/MISO1), U4.2 (MISO/DO)
- new net MOSI: U1.33 (PA7/ADC7/MOSI1), U4.5 (MOSI/DI)
- new net S0: U1.5 (PA8), U3.10 (S0)
- new net S1: U1.6 (PA9/TX1), U3.11 (S1)
- new net S2: U1.7 (PA10/RX1), U3.14 (S2)
- new net S3: U1.10 (PA15), U3.13 (S3)
- new net SIG: U1.27 (PA1/ADC1), U3.1 (COM)
- no-connect marks 32 -> 8
Other:
- note added: "5V DC Input"
- note added: "FLASH MEMORY"
- note added: "MUX"
- note added: "STM32F411CEU6 Blackpill"
- note removed: "5V DC in"
- note removed: "teensy"
- moved on the sheet: C1, C10, C11, C2, C3, C4, C5, C6, C7, C8, C9, J1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
