File: MC8P_MIDI_CONTROLLER_KiCad/MC8P_MIDI_CONTROLLER/MC8P_MIDI_CONTROLLER.kicad_pcb (KiCad board)
At the start: 2 copper layers, 155 x 288 mm, 61 parts, among them J1 MIDI OUT, J2 5V, SW1 ASSIGN, SW2 ENTER, SW3 PREV, SW4 NEXT, U1 Teensy4.0

Commit message: Black Pill Schematic & PCB
Parts:
- removed the ? at (169.0, 210.0)
- removed the ? at (169.0, 290.0)
- removed the ? at (26.0, 210.0)
- removed the ? at (169.0, 198.0)
- removed the ? at (26.0, 290.0)
- removed the ? at (26.0, 198.0)
- removed the ? at (26.0, 106.0)
- removed the ? at (169.0, 118.0)
- removed the ? at (26.0, 118.0)
- removed the G*** at (122.0, 229.1) (x2)
- removed the G*** at (112.5, 224.8)
- removed the REF** at (83.0, 161.3)
- removed the REF** at (106.0, 185.2)
- removed the REF** at (26.0, 26.0)
- removed the REF** at (106.0, 161.3)
- removed the REF** at (83.0, 185.2)
- removed the REF** at (169.0, 106.0)
- removed the REF** at (169.0, 26.0)
- removed the REF** at (60.0, 185.2)
- removed the REF** at (60.0, 161.3)
- removed the REF** at (37.0, 185.2)
- removed the REF** at (37.0, 161.3)
- added ?: , , F.Cu at (167.2, 120.5)
- added ?: , , F.Cu at (167.3, 212.5)
- added ?: , , F.Cu at (24.2, 108.5)
- added ?: , , F.Cu at (24.2, 120.5)
- added ?: , , F.Cu at (167.2, 200.5)
- added ?: , , F.Cu at (167.3, 292.5)
- added ?: , , F.Cu at (24.3, 212.5)
- added ?: , , F.Cu at (24.2, 200.5)
- added ?: , , F.Cu at (24.3, 292.5)
- added C13: 100nF_0603_16V, Capacitor_SMD:C_1206_3216Metric, F.Cu at (80.8, 30.8)
- added C14: 100nF_0603_16V, Capacitor_SMD:C_1206_3216Metric, F.Cu at (134.8, 33.5)
- added C15: 100nF_0603_16V, Capacitor_SMD:C_1206_3216Metric, F.Cu at (68.5, 68.9)
- added C16: 10uF, Capacitor_SMD:C_1206_3216Metric_Pad1.33x1.80mm_HandSolder, F.Cu at (71.0, 68.9)
- added D1: LED, LED_SMD:LED_1206_3216Metric_Pad1.42x1.75mm_HandSolder, F.Cu at (43.0, 53.8)
- added D2: BAT43, Diode_SMD:D_SOD-123, F.Cu at (70.0, 64.5)
- added G***: LOGO, MC8P_BITMAP_FOOTPRINTS:MC8P_PXLART_SPACE_FMASK_45X40, F.Cu at (110.8, 227.2)
- added G*** (x2): LOGO, MC8P_BITMAP_FOOTPRINTS:MC8P_PXLART_SPACE_FMASK_45X40, F.Cu at (120.3, 231.6)
- added R7: 10k_0402, PCM_4ms_Resistor:R_0603, F.Cu at (94.2, 29.5)
- added R8: 10k_0402, PCM_4ms_Resistor:R_0603, F.Cu at (42.2, 51.0)
- added REF**: Panel Knob 2P, SimpleSynthPanel:Panel Knob 2P, F.Cu at (58.3, 187.7)
- added REF**: MountingHole_M3_Standoff, DIYSynthMNL:MountingHole_M3_Standoff, F.Cu at (167.2, 28.5)
- added REF**: Panel Knob 2P, SimpleSynthPanel:Panel Knob 2P, F.Cu at (35.3, 163.8)
- added REF**: Panel Knob 2P, SimpleSynthPanel:Panel Knob 2P, F.Cu at (104.3, 163.8)
- added REF**: Panel Knob 2P, SimpleSynthPanel:Panel Knob 2P, F.Cu at (81.2, 163.8)
- added REF**: Panel Knob 2P, SimpleSynthPanel:Panel Knob 2P, F.Cu at (104.3, 187.7)
- added REF**: Panel Knob 2P, SimpleSynthPanel:Panel Knob 2P, F.Cu at (58.2, 163.8)
- added REF**: Panel Knob 2P, SimpleSynthPanel:Panel Knob 2P, F.Cu at (35.3, 187.7)
- added REF**: Panel Knob 2P, SimpleSynthPanel:Panel Knob 2P, F.Cu at (81.3, 187.7)
- added REF**: MountingHole_M3_Standoff, DIYSynthMNL:MountingHole_M3_Standoff, F.Cu at (24.2, 28.5)
- added REF**: MountingHole_M3_Standoff, DIYSynthMNL:MountingHole_M3_Standoff, F.Cu at (167.2, 108.5)
- added U3: CD74HC4067M, Package_SO:SOIC-24W_7.5x15.4mm_P1.27mm, F.Cu at (89.8, 37.2)
- added U4: W25Q64, Package_SO:SOIC-8_3.9x4.9mm_P1.27mm, F.Cu at (37.1, 47.9)
- C1, C2, C3, C4, C5, C6, C7, C8: footprint Capacitor_THT:C_Axial_L3.8mm_D2.6mm_P7.50mm_Horizontal -> Capacitor_SMD:C_1206_3216Metric_Pad1.33x1.80mm_HandSolder
- C10, C9: footprint Capacitor_THT:C_Disc_D5.0mm_W2.5mm_P5.00mm -> Capacitor_SMD:C_1206_3216Metric_Pad1.33x1.80mm_HandSolder
- C12: value 10uF_4x5.3_10V -> 100nF_0603_16V; footprint Capacitor_THT:CP_Radial_D4.0mm_P1.50mm -> Capacitor_SMD:C_1206_3216Metric
- J1: moved to B.Cu
- J2: value 5V -> Jack-DC
- R1, R2, R3, R4: value 10k_0402 -> 10k; footprint PCM_4ms_Resistor:R_Axial_DIN0207_L6.3mm_D2.5mm_P7.62mm_Horizontal -> PCM_4ms_Resistor:R_0603
- R5, R6: footprint PCM_4ms_Resistor:R_Axial_DIN0207_L6.3mm_D2.5mm_P7.62mm_Horizontal -> PCM_4ms_Resistor:R_0603
- U1: value Teensy4.0 -> ~; footprint teensy:Teensy40 -> blackpill:Z_module_black_pill_STM32F411; moved to B.Cu
- moved C5 80.6 mm to (37.2, 85.5), turned to 0 degrees
- moved C12 78.8 mm to (37.6, 53.1), turned to 0 degrees
- moved C6 56.7 mm to (59.8, 85.8), turned to 0 degrees
- moved C11 52.8 mm to (56.0, 28.2), turned to 0 degrees
- moved C10 45.7 mm to (57.5, 34.8), turned to 0 degrees
- moved C9 40.8 mm to (57.5, 32.0), turned to 0 degrees
- moved C1 40.1 mm to (36.8, 61.5), turned to 0 degrees
- moved C7 37.3 mm to (82.8, 85.5), turned to 0 degrees
- moved C8 33.9 mm to (105.7, 85.5), turned to 0 degrees
- moved R4 31.4 mm to (119.5, 71.2)
- moved R3 25.6 mm to (119.5, 69.5)
- moved C2 22.9 mm to (59.8, 61.5), turned to 0 degrees
- moved R2 18.2 mm to (119.5, 66.0)
- moved C4 17.4 mm to (106.0, 61.8), turned to 0 degrees
- moved R1 15.9 mm to (119.5, 67.8)
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Connections:
- C1 pad 1: A0 -> pot1
- C12 pad 1: 5V -> GND
- C12 pad 2: GND -> 3V3
- C2 pad 1: A1 -> pot2
- C3 pad 1: A2 -> pot3
- C4 pad 1: A3 -> pot4
- C5 pad 1: A9 -> pot5
- C6 pad 1: A8 -> pot6
- C7 pad 1: A7 -> pot7
- C8 pad 1: A6 -> pot8
- J2 pad 1: 5V -> Net-(D2-A)
- J2 pad 3: GND -> (no net)
- R1 pad 1: D5 -> ASSIGN
- R2 pad 1: D6 -> ENTER
- R3 pad 1: D7 -> PREV
- R4 pad 1: D8 -> NEXT
- R6 pad 1: Vcc -> 3V3
- RV1 pad 2: A0 -> pot1
- RV2 pad 2: A1 -> pot2
- RV3 pad 2: A2 -> pot3
- RV4 pad 2: A3 -> pot4
- RV5 pad 2: A6 -> pot5
- RV6 pad 2: A7 -> pot6
- RV7 pad 2: A8 -> pot7
- RV8 pad 2: A9 -> pot8
- SW1 pad 2: D5 -> ASSIGN
- SW2 pad 2: D6 -> ENTER
- SW3 pad 2: D7 -> PREV
- SW4 pad 2: D8 -> NEXT
- U1 pad 1: GND -> ASSIGN
- U1 pad 10: D8 -> S3
- U1 pad 14: unconnected-(U1-12_MISO_MQSL-Pad14) -> SCL0
- U1 pad 15: unconnected-(U1-VBAT-Pad15) -> SDA0
- U1 pad 17: GND -> unconnected-(U1-1PB9-Pad17)
- U1 pad 18: unconnected-(U1-PROGRAM-Pad18) -> Vcc
- U1 pad 19: unconnected-(U1-ON_OFF-Pad19) -> GND
- U1 pad 2: unconnected-(U1-0_RX1_CRX2_CS1-Pad2) -> ENTER
- U1 pad 20: unconnected-(U1-13_SCK_CRX1_LED-Pad20) -> 3V3
- U1 pad 21: A0 -> unconnected-(U1-VBAT-Pad21)
- U1 pad 22: A1 -> unconnected-(U1-PC13-Pad22)
- U1 pad 23: A2 -> unconnected-(U1-PC14-Pad23)
- U1 pad 24: A3 -> unconnected-(U1-PC15-Pad24)
- U1 pad 25: SDA0 -> unconnected-(U1-RESET-Pad25)
- U1 pad 26: SCL0 -> unconnected-(U1-PA0/ADC0-Pad26)
- U1 pad 27: A6 -> SIG
- U1 pad 28: A7 -> TX0
- U1 pad 29: A8 -> unconnected-(U1-PA3/ADC3/RX2-Pad29)
- U1 pad 3: TX0 -> PREV
- U1 pad 30: A9 -> CS
- U1 pad 31: 3V3 -> CLK
- U1 pad 32: GND -> MISO
- U1 pad 33: 5V -> MOSI
- U1 pad 34: Vcc -> unconnected-(U1-PB0/ADC8-Pad34)
- U1 pad 38: unconnected-(U1-27_A13_SCK1-Pad38) -> 3V3
- U1 pad 39: unconnected-(U1-28_RX7-Pad39) -> GND
- U1 pad 4: unconnected-(U1-2_OUT2-Pad4) -> NEXT
- U1 pad 40: unconnected-(U1-29_TX7-Pad40) -> Vcc
- U1 pad 5: unconnected-(U1-3_LRCLK2-Pad5) -> S0
- U1 pad 6: unconnected-(U1-4_BCLK2-Pad6) -> S1
- U1 pad 7: D5 -> S2
- U1 pad 8: D6 -> unconnected-(U1-PA11-Pad8)
- U1 pad 9: D7 -> unconnected-(U1-PA12-Pad9)
Routing:
- net D5: track 278.5 -> 0.00 mm
- net D7: track 257.8 -> 0.00 mm
- net D6: track 252.4 -> 0.00 mm
- net D8: track 250.9 -> 0.00 mm
- net NEXT: track 0.00 -> 208.8 mm, vias 0 -> 1
- net PREV: track 0.00 -> 198.1 mm, vias 0 -> 1
- net A6: track 158.7 -> 0.00 mm
- net Net-(D2-A): track 0.00 -> 157.3 mm, vias 0 -> 1
- net pot1: track 0.00 -> 155.2 mm, vias 0 -> 1
- net ENTER: track 0.00 -> 148.3 mm, vias 0 -> 1
- net pot5: track 0.00 -> 141.4 mm, vias 0 -> 2
- net A7: track 136.6 -> 0.00 mm
- net pot2: track 0.00 -> 135.0 mm, vias 0 -> 3
- net pot6: track 0.00 -> 124.2 mm, vias 0 -> 2
- net A8: track 115.3 -> 0.00 mm
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
Commit message: updated BOM
Parts:
- removed the G*** at (85.8, 226.0)
- removed the G*** at (156.0, 292.5)
